Commit message: updating urdf to use yellowstone definition from ologic project tango

File: src/head_unit/urdf/head_unit.urdf (robot description, URDF)
Before this commit: robot head_unit, 5 links, 5 joints
Links:
- removed link depth_camera
- removed link fisheye_camera
- removed link fix
- removed link imu
- link head_unit: geometry visual mesh filename=package://head_unit/urdf/tango_yellowstone.dae scale=0.01 0.01 0.01
Joints:
- removed joint head_unit_to_depth_camera
- removed joint head_unit_to_fisheye_camera
- removed joint head_unit_to_fix
- removed joint head_unit_to_imu

File: src/head_unit/urdf/head_unit.xacro (robot description, xacro)
@@ -1,2 +1,24 @@
+<?xml version="1.0"?>
+<robot xmlns:xacro="http://www.ros.org/wiki/xacro" name="head_unit">
+  <link name="head_unit">
+    <visual>
+      <!-- <origin xyz="0 0 0" rpy="3.14 0 1.57 " /> -->
+      <origin xyz="-1.0 -1.0 0" rpy="0 0 0" /> -->
+      <geometry>
+        <mesh filename="package://head_unit/urdf/tango_yellowstone.dae"
+          scale="0.01 0.01 0.01" />
+      </geometry>
+      <material name="grey">
+        <color rgba="0.1 0.1 .5 1"/>
+      </material>
+    </visual>
+  </link>
+  <joint name="base_link_to_head_unit" type="fixed">
+    <parent link="base_link" />
+    <child link="head_unit" />
+    <origin xyz="0 0 1.2192" rpy="0 0 0" />
+  </joint>
+</robot>
+<!--
 <?xml version="1.0"?>
 <robot xmlns:xacro="http://www.ros.org/wiki/xacro" name="head_unit">
@@ -17,5 +39,4 @@
     <origin xyz="0 0 1.2192" rpy="0 0 0" />
   </joint>
-  <!-- IMU -->
   <link name="imu">
     <visual>
@@ -33,5 +54,4 @@
     <origin xyz="0 0 0" rpy="0 0 0" />
   </joint>
-  <!-- GPS UNIT -->
   <link name="fix">
     <visual>
@@ -79,7 +99,5 @@
     <origin xyz="0 0.4 0" rpy="0 0 0" />
   </joint>
-<!--
 <node pkg="tf" type="static_transform_publisher" name="device_to_depth_cam" args="0 0 0 0 0.24 0 device depth_camera 10"/>
 <node pkg="tf" type="static_transform_publisher" name="fisheye_to_depth_cam" args="0 -0.05 0 0 0 0 depth_camera fisheye_camera 10"/>
 -->
-</robot>

File: src/navbot/urdf/navbot.urdf (robot description, URDF)
Before this commit: robot blah, 20 links, 19 joints
Links:
- removed link depth_camera
- removed link fisheye_camera
- removed link fix
- removed link imu
- link head_unit: geometry visual mesh filename=package://head_unit/urdf/tango_yellowstone.dae scale=0.01 0.01 0.01
Joints:
- removed joint head_unit_to_depth_camera
- removed joint head_unit_to_fisheye_camera
- removed joint head_unit_to_fix
- removed joint head_unit_to_imu

Commit message: updating urdf files for tango placement

File: src/head_unit/urdf/head_unit.urdf (robot description, URDF)
Before this commit: robot head_unit, 1 links, 1 joints
Links:
- added link phone; visual mesh filename=package://head_unit/urdf/tango_yellowstone.dae scale=0.01 0.01 0.01
- added link unity; visual box size=0.0001 0.0001 0.0001
- link head_unit: geometry visual box size=0.0160528 0.1992376 0.119888
Joints:
- added joint base_link_to_unity: type fixed, parent base_link, child unity, origin xyz=0 0 0 rpy=0 0 0
- added joint unity_to_phone: type fixed, parent unity, child phone, origin xyz=0 0 0 rpy=0 0 0

File: src/head_unit/urdf/head_unit.xacro (robot description, xacro)
@@ -3,9 +3,7 @@
   <link name="head_unit">
     <visual>
-      <!-- <origin xyz="0 0 0" rpy="3.14 0 1.57 " /> -->
-      <origin xyz="-1.0 -1.0 0" rpy="0 0 0" /> -->
+      <origin xyz="-1.0 -1.0 0" rpy="0 0 0" />
       <geometry>
-        <mesh filename="package://head_unit/urdf/tango_yellowstone.dae"
-          scale="0.01 0.01 0.01" />
+        <box size="0.0160528 0.1992376 0.119888"/>
       </geometry>
       <material name="grey">
@@ -19,4 +17,45 @@
     <origin xyz="0 0 1.2192" rpy="0 0 0" />
   </joint>
+  <link name="phone">
+    <visual>
+      <!-- <origin xyz="0 0 0" rpy="3.14 0 1.57 " /> -->
+      <origin xyz="-1.0 -1.0 0" rpy="0 0 0" />
+      <geometry>
+        <mesh filename="package://head_unit/urdf/tango_yellowstone.dae"
+          scale="0.01 0.01 0.01" />
+      </geometry>
+      <material name="grey">
+        <color rgba="0.1 0.1 .5 1"/>
+      </material>
+    </visual>
+  </link>
+  <link name="unity">
+    <visual>
+      <origin xyz="0 0 0" rpy="0 0 0" />
+      <geometry>
+        <box size="0.0001 0.0001 0.0001"/>
+      </geometry>
+      <material name="grey">
+        <color rgba="0.1 0.1 .5 1"/>
+      </material>
+    </visual>
+  </link>
+  <joint name="unity_to_phone" type="fixed">
+    <parent link="unity" />
+    <child link="phone" />
+    <origin xyz="0 0 0" rpy="0 0 0" />
+  </joint>
+  <joint name="base_link_to_unity" type="fixed">
+    <parent link="base_link" />
+    <child link="unity" />
+    <origin xyz="0 0 0" rpy="0 0 0" />
+  </joint>
+<!--
+  <joint name="head_unit_to_phone" type="fixed">
+    <parent link="head_unit" />
+    <child link="phone" />
+    <origin xyz="0 0 0" rpy="0 0 0" />
+  </joint>
+-->
 </robot>
 <!--

File: src/navbot/urdf/navbot.urdf (robot description, URDF)
Before this commit: robot blah, 16 links, 15 joints
Links:
- added link phone; visual mesh filename=package://head_unit/urdf/tango_yellowstone.dae scale=0.01 0.01 0.01
- added link unity; visual box size=0.0001 0.0001 0.0001
- link head_unit: geometry visual box size=0.0160528 0.1992376 0.119888
Joints:
- added joint base_link_to_unity: type fixed, parent base_link, child unity, origin xyz=0 0 0 rpy=0 0 0
- added joint unity_to_phone: type fixed, parent unity, child phone, origin xyz=0 0 0 rpy=0 0 0

Commit message: Adding Michael's head unit urdf changes.

File: src/head_unit/urdf/head_unit.urdf (robot description, URDF)
Before this commit: robot head_unit, 3 links, 3 joints
Links:
- link phone: geometry visual mesh filename=package://head_unit/urdf/tango_yellowstone.dae scale=0.001 0.001 0.001
Joints:
- removed joint base_link_to_unity
- added joint head_unit_to_unity: type fixed, parent head_unit, child unity, origin xyz=0.1 0.1 0 rpy=1.22 0 -1.57
- joint base_link_to_head_unit: origin xyz=0 0 1.2192 rpy=0 0 0 -> xyz=0 0 0.12 rpy=0 0 0

File: src/head_unit/urdf/head_unit.xacro (robot description, xacro)
@@ -3,5 +3,5 @@
   <link name="head_unit">
     <visual>
-      <origin xyz="-1.0 -1.0 0" rpy="0 0 0" />
+      <origin xyz="0 0 0" rpy="0 0 0" />
       <geometry>
         <box size="0.0160528 0.1992376 0.119888"/>
@@ -12,16 +12,23 @@
     </visual>
   </link>
+  <!--
+  <joint name="platform_upper_to_head_unit" type="fixed">
+    <parent link="base_link" />
+    <child link="platform_upper" />
+    <origin xyz="0 0 0" rpy="0 0 0" />
+  </joint>
+  -->
   <joint name="base_link_to_head_unit" type="fixed">
     <parent link="base_link" />
     <child link="head_unit" />
-    <origin xyz="0 0 1.2192" rpy="0 0 0" />
+    <origin xyz="0 0 0.12" rpy="0 0 0" />
   </joint>
   <link name="phone">
     <visual>
       <!-- <origin xyz="0 0 0" rpy="3.14 0 1.57 " /> -->
-      <origin xyz="-1.0 -1.0 0" rpy="0 0 0" />
+      <!-- <origin xyz="0 0 0" rpy="1.22 0 1.57" /> -->
       <geometry>
         <mesh filename="package://head_unit/urdf/tango_yellowstone.dae"
-          scale="0.01 0.01 0.01" />
+          scale="0.001 0.001 0.001" />
       </geometry>
       <material name="grey">
@@ -32,5 +39,5 @@
   <link name="unity">
     <visual>
-      <origin xyz="0 0 0" rpy="0 0 0" />
+      <!-- <origin xyz="0 0 0" rpy="0 0 0" /> -->
       <geometry>
         <box size="0.0001 0.0001 0.0001"/>
@@ -46,8 +53,8 @@
     <origin xyz="0 0 0" rpy="0 0 0" />
   </joint>
-  <joint name="base_link_to_unity" type="fixed">
-    <parent link="base_link" />
+  <joint name="head_unit_to_unity" type="fixed">
+    <parent link="head_unit" />
     <child link="unity" />
-    <origin xyz="0 0 0" rpy="0 0 0" />
+    <origin xyz="0.1 0.1 0" rpy="1.22 0 -1.57" />
   </joint>
 <!--

File: src/navbot/urdf/navbot.urdf (robot description, URDF)
Before this commit: robot blah, 18 links, 17 joints
Links:
- link phone: geometry visual mesh filename=package://head_unit/urdf/tango_yellowstone.dae scale=0.001 0.001 0.001
Joints:
- removed joint base_link_to_unity
- added joint head_unit_to_unity: type fixed, parent head_unit, child unity, origin xyz=0.1 0.1 0 rpy=1.22 0 -1.57
- joint base_link_to_head_unit: origin xyz=0 0 1.2192 rpy=0 0 0 -> xyz=0 0 0.12 rpy=0 0 0

Commit message: Adding structure sensor ir and stereo camera to head_unit xacro

File: src/head_unit/urdf/head_unit.urdf (robot description, URDF)
Before this commit: robot head_unit, 3 links, 3 joints
Links:
- added link camera_left; visual box size=0.0001 0.0001 0.0001
- added link camera_right; visual box size=0.0001 0.0001 0.0001
- added link structure_ir; visual box size=0.0001 0.0001 0.0001
Joints:
- added joint head_unit_to_camera_left: type fixed, parent head_unit, child camera_left, origin xyz=0 -0.0177 0.381 rpy=0 0 0
- added joint head_unit_to_camera_right: type fixed, parent head_unit, child camera_right, origin xyz=0 0.0177 0.381 rpy=0 0 0
- added joint head_unit_to_structure_ir: type fixed, parent head_unit, child structure_ir, origin xyz=0 0.0457 0.0813 rpy=0 0 0
