Commit message: update kinect xacro and main navbot mkii urdf to show the kinect properly

File: src/head_unit/urdf/kinect2.xacro (robot description, xacro)
@@ -13,11 +13,10 @@
       <origin rpy="${rpy}" xyz="${xyz}" />
       <parent link="${parent}"/>
-      <child link="${prefix}_kinect2_rgb_optical_frame"/>
+      <child link="kinect2_link"/>
     </joint>
-    <link name="${prefix}_kinect2_rgb_optical_frame">
+   <link name="kinect2_link">
       <visual>
         <origin rpy="0 0 0" xyz="0 0 0"/>
         <geometry>
-          <!-- these meshes were exported in mm, so scale back to m -->
           <mesh filename="package://head_unit/urdf/meshes/kinect2_origin_on_rgb_optical_frame.stl" scale="0.001 0.001 0.001"/>
         </geometry>
@@ -25,5 +24,17 @@
       </visual>
     </link>
+<!--
+    <link name="kinect2_rgb_optical_frame">
+      <visual>
+        <origin rpy="0 0 0" xyz="0 0 0"/>
+        <geometry>
+          <mesh filename="package://head_unit/urdf/meshes/kinect2_origin_on_rgb_optical_frame.stl" scale="0.001 0.001 0.001"/>
+        </geometry>
+        <material name="Kinect2Grey"/>
+      </visual>
+    </link>
+-->
   </xacro:macro>
-  <xacro:kinect2_xacro prefix="head_unit" parent="head_unit" rpy="0 0 ${pi/2}" xyz="0 0.108 0.07" />
+  <xacro:kinect2_xacro prefix="head_unit" parent="head_unit" rpy="${-pi/2} 0 ${-pi/2}" xyz="0.04 -0.098 0.035" />
+ <!--  <xacro:kinect2_xacro prefix="head_unit" parent="head_unit" rpy="0 0 ${pi/2}" xyz="0 0.108 0.07" /> -->
 </robot>

File: src/navbot/urdf/navbot_mkii.urdf (robot description, URDF)
Before this commit: robot blah, 9 links, 8 joints
Links:
- removed link head_unit_kinect2_rgb_optical_frame
- added link kinect2_link; visual mesh filename=package://head_unit/urdf/meshes/kinect2_origin_on_rgb_optic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 scale=0.001 0.001 0.001
Joints:
- joint head_unit_kinect2_in_joint: child head_unit_kinect2_rgb_optical_frame -> kinect2_link; origin xyz=0 0.108 0.07 rpy=0 0 1.5707963268 -> xyz=0.04 -0.098 0.035 rpy=-1.5707963268 0 -1.5707963268

Commit message: updating xacro and rdf to get the laser scan and point clouds lined up correctly by setting a transform for camera_depth_frame

File: src/head_unit/urdf/kinect2.xacro (robot description, xacro)
@@ -24,4 +24,17 @@
       </visual>
     </link>
+    <joint name="kinect2_link_to_camera_depth_frame" type="fixed">
+      <origin rpy="${pi/2} ${-pi/2} 0" xyz="0 0 0" />
+      <parent link="kinect2_link"/>
+      <child link="camera_depth_frame"/>
+    </joint>
+   <link name="camera_depth_frame">
+      <visual>
+        <origin rpy="0 0 0" xyz="0 0 0"/>
+        <geometry>
+          <box size="0.001 0.001 0.001" />
+        </geometry>
+      </visual>
+    </link>
 <!--
     <link name="kinect2_rgb_optical_frame">

File: src/navbot/urdf/navbot_mkii.urdf (robot description, URDF)
Before this commit: robot blah, 9 links, 8 joints
Links:
- added link camera_depth_frame; visual box size=0.001 0.001 0.001
Joints:
- added joint kinect2_link_to_camera_depth_frame: type fixed, parent kinect2_link, child camera_depth_frame, origin xyz=0 0 0 rpy=1.5707963268 -1.5707963268 0
