Commit message: Added t-slot rod and brackets to xacro

File: src/head_unit/urdf/head_unit_mkii.xacro (robot description, xacro)
@@ -1,9 +1,10 @@
 <?xml version="1.0"?>
-<robot xmlns:xacro="http://www.ros.org/wiki/xacro" name="head_unit">
+<robot xmlns:xacro="http://www.ros.org/wiki/xacro" name="head_unit">i
+  <xacro:property name="pi" value="3.14159265359" />
   <link name="head_unit">
     <visual>
       <origin xyz="0 0 0" rpy="0 0 0" />
       <geometry>
-        <box size="0.0677 0.1120 0.0200"/>
+        <box size="0.0677 0.1120 0.0200" />
       </geometry>
       <material name="grey">
@@ -17,4 +18,54 @@
     <origin xyz="0 0 1.2192" rpy="0 0 0" />
   </joint>
+  <link name="head_mount">
+    <visual>
+      <origin xyz="0 0 0" rpy="0 0 0" />
+      <geometry>
+        <box size="0.1268 0.1525 0.0096" />
+      </geometry>
+      <material name="silver">
+        <color rgba="129 129 129 1" />
+      </material>
+    </visual>
+  </link>
+  <joint name="head_unit_to_head_mount" type="fixed">
+    <parent link="head_unit" />
+    <child link="head_mount" />
+    <origin xyz="0 0 -0.94" rpy="0 0 0 " />
+  </joint>
+  <link name="t-slot-rod">
+    <visual>
+      <origin xyz="0 0 0" rpy="0 0 0" />
+      <geometry>
+         <mesh filename="package://head_unit/urdf/meshes/t-slot-rod.stl" scale="1 1 0.8"/>
+      </geometry>
+      <material name="silver" />
+    </visual>
+  </link>
+  <joint name="head_unit_to_t-slot-rod" type="fixed">
+    <parent link="head_unit" />
+    <child link="t-slot-rod" />
+    <origin xyz="0 0 -0.49" rpy="0 0 0" />
+  </joint>
+  <xacro:macro name="t-slot-bracket" params="name xyz rpy">
+    <link name="t-slot-bracket-${name}">
+      <visual>
+        <origin xyz="0 0 0" rpy="0 0 0" />
+        <geometry>
+           <mesh filename="package://head_unit/urdf/meshes/t-slot-bracket.stl" scale="1 1 1"/>
+        </geometry>
+        <material name="silver" />
+      </visual>
+    </link>
+    <joint name="head_unit_to_t-slot-bracket-${name}" type="fixed">
+      <parent link="head_unit" />
+      <child link="t-slot-bracket-${name}" />
+      <origin xyz="${xyz}" rpy="${rpy}" />
+    </joint>
+  </xacro:macro>
+  <xacro:t-slot-bracket name="bottom-left" xyz="0 0.0191 -0.935" rpy="${pi/2} 0 ${pi/2}" />
+  <xacro:t-slot-bracket name="bottom-right" xyz="0 -0.0191 -0.935" rpy="${pi/2} 0 -${pi/2}" />
+  <xacro:t-slot-bracket name="top-left" xyz="0 0.0191 -0.01" rpy="-${pi/2} 0 ${pi/2}" />
+  <xacro:t-slot-bracket name="top-right" xyz="0 -0.0191 -0.01" rpy="-${pi/2} 0 -${pi/2}" />
   <xacro:include filename="../../head_unit/urdf/kinect2.xacro" />
 </robot>

File: src/navbot/urdf/navbot_mkii.urdf (robot description, URDF)
Before this commit: robot blah, 3 links, 2 joints
Links:
- added link head_mount; visual box size=0.1268 0.1525 0.0096
- added link t-slot-bracket-bottom-left; visual mesh filename=package://head_unit/urdf/meshes/t-slot-bracket.stl scale=1 1 1
- added link t-slot-bracket-bottom-right; visual mesh filename=package://head_unit/urdf/meshes/t-slot-bracket.stl scale=1 1 1
- added link t-slot-bracket-top-left; visual mesh filename=package://head_unit/urdf/meshes/t-slot-bracket.stl scale=1 1 1
- added link t-slot-bracket-top-right; visual mesh filename=package://head_unit/urdf/meshes/t-slot-bracket.stl scale=1 1 1
- added link t-slot-rod; visual mesh filename=package://head_unit/urdf/meshes/t-slot-rod.stl scale=1 1 0.8
Joints:
- added joint head_unit_to_head_mount: type fixed, parent head_unit, child head_mount, origin xyz=0 0 -0.94 rpy=0 0 0 
- added joint head_unit_to_t-slot-bracket-bottom-left: type fixed, parent head_unit, child t-slot-bracket-bottom-left, origin xyz=0 0.0191 -0.935 rpy=1.5707963268 0 1.5707963268
- added joint head_unit_to_t-slot-bracket-bottom-right: type fixed, parent head_unit, child t-slot-bracket-bottom-right, origin xyz=0 -0.0191 -0.935 rpy=1.5707963268 0 -1.5707963268
- added joint head_unit_to_t-slot-bracket-top-left: type fixed, parent head_unit, child t-slot-bracket-top-left, origin xyz=0 0.0191 -0.01 rpy=-1.5707963268 0 1.5707963268
- added joint head_unit_to_t-slot-bracket-top-right: type fixed, parent head_unit, child t-slot-bracket-top-right, origin xyz=0 -0.0191 -0.01 rpy=-1.5707963268 0 -1.5707963268
- added joint head_unit_to_t-slot-rod: type fixed, parent head_unit, child t-slot-rod, origin xyz=0 0 -0.49 rpy=0 0 0

Commit message: Adding project tango to head unit mk ii.

File: src/head_unit/urdf/head_unit_mkii.xacro (robot description, xacro)
@@ -69,3 +69,4 @@
   <xacro:t-slot-bracket name="top-right" xyz="0 -0.0191 -0.01" rpy="-${pi/2} 0 -${pi/2}" />
   <xacro:include filename="../../head_unit/urdf/kinect2.xacro" />
+  <xacro:include filename="../../head_unit/urdf/project_tango.xacro" />
 </robot>

File: src/navbot/urdf/navbot_mkii.urdf (robot description, URDF)
Before this commit: robot blah, 10 links, 9 joints
Links:
- added link phone; visual mesh filename=package://head_unit/urdf/tango_yellowstone.dae scale=0.001 0.001 0.001
- added link unity; visual box size=0.0001 0.0001 0.0001
Joints:
- added joint head_unit_to_unity: type fixed, parent head_unit, child unity, origin xyz=0 -0.1 -0.1 rpy=1.22 0 -1.5707963268
- added joint unity_to_phone: type fixed, parent unity, child phone, origin xyz=0 0 0 rpy=0 0 0

Commit message: Tuning xacro for project tango

File: src/head_unit/urdf/head_unit_mkii.xacro (robot description, xacro)
@@ -16,5 +16,5 @@
     <parent link="base_link" />
     <child link="head_unit" />
-    <origin xyz="0 0 1.2192" rpy="0 0 0" />
+    <origin xyz="0 0 0.45" rpy="0 0 0" /> <!-- fix height -->
   </joint>
   <link name="head_mount">
@@ -32,5 +32,5 @@
     <parent link="head_unit" />
     <child link="head_mount" />
-    <origin xyz="0 0 -0.94" rpy="0 0 0 " />
+    <origin xyz="0 0 -0.2159" rpy="0 0 0 " />
   </joint>
   <link name="t-slot-rod">
@@ -38,5 +38,5 @@
       <origin xyz="0 0 0" rpy="0 0 0" />
       <geometry>
-         <mesh filename="package://head_unit/urdf/meshes/t-slot-rod.stl" scale="1 1 0.8"/>
+         <mesh filename="package://head_unit/urdf/meshes/t-slot-rod.stl" scale="1 1 0.2"/>
       </geometry>
       <material name="silver" />
@@ -46,5 +46,5 @@
     <parent link="head_unit" />
     <child link="t-slot-rod" />
-    <origin xyz="0 0 -0.49" rpy="0 0 0" />
+    <origin xyz="0 0 -0.1065" rpy="0 0 0" />
   </joint>
   <xacro:macro name="t-slot-bracket" params="name xyz rpy">
@@ -64,6 +64,6 @@
     </joint>
   </xacro:macro>
-  <xacro:t-slot-bracket name="bottom-left" xyz="0 0.0191 -0.935" rpy="${pi/2} 0 ${pi/2}" />
-  <xacro:t-slot-bracket name="bottom-right" xyz="0 -0.0191 -0.935" rpy="${pi/2} 0 -${pi/2}" />
+  <xacro:t-slot-bracket name="bottom-left" xyz="0 0.0191 -0.135" rpy="${pi/2} 0 ${pi/2}" />
+  <xacro:t-slot-bracket name="bottom-right" xyz="0 -0.0191 -0.135" rpy="${pi/2} 0 -${pi/2}" />
   <xacro:t-slot-bracket name="top-left" xyz="0 0.0191 -0.01" rpy="-${pi/2} 0 ${pi/2}" />
   <xacro:t-slot-bracket name="top-right" xyz="0 -0.0191 -0.01" rpy="-${pi/2} 0 -${pi/2}" />

File: src/head_unit/urdf/project_tango.xacro (robot description, xacro)
@@ -31,5 +31,5 @@
     <parent link="head_unit" />
     <child link="unity" />
-    <origin xyz="0 -0.1 -0.1" rpy="1.22 0 ${-pi/2}" />
+    <origin xyz="-0.15 0.1 -0.185" rpy="1.22 0 ${-pi/2}" />
   </joint>
 </robot>

File: src/navbot/urdf/navbot_mkii.urdf (robot description, URDF)
Before this commit: robot blah, 12 links, 11 joints
Links:
- link t-slot-rod: geometry visual mesh filename=package://head_unit/urdf/meshes/t-slot-rod.stl scale=1 1 0.2
Joints:
- joint base_link_to_head_unit: origin xyz=0 0 1.2192 rpy=0 0 0 -> xyz=0 0 0.45 rpy=0 0 0
- joint head_unit_to_head_mount: origin xyz=0 0 -0.94 rpy=0 0 0  -> xyz=0 0 -0.2159 rpy=0 0 0 
- joint head_unit_to_t-slot-bracket-bottom-left: origin xyz=0 0.0191 -0.935 rpy=1.5707963268 0 1.5707963268 -> xyz=0 0.0191 -0.135 rpy=1.5707963268 0 1.5707963268
- joint head_unit_to_t-slot-bracket-bottom-right: origin xyz=0 -0.0191 -0.935 rpy=1.5707963268 0 -1.5707963268 -> xyz=0 -0.0191 -0.135 rpy=1.5707963268 0 -1.5707963268
- joint head_unit_to_t-slot-rod: origin xyz=0 0 -0.49 rpy=0 0 0 -> xyz=0 0 -0.1065 rpy=0 0 0
- joint head_unit_to_unity: origin xyz=0 -0.1 -0.1 rpy=1.22 0 -1.5707963268 -> xyz=-0.15 0.1 -0.185 rpy=1.22 0 -1.5707963268

Commit message: Fixed xacro for mk ii

File: src/head_unit/urdf/head_unit_mkii.xacro (robot description, xacro)
@@ -1,4 +1,4 @@
 <?xml version="1.0"?>
-<robot xmlns:xacro="http://www.ros.org/wiki/xacro" name="head_unit">i
+<robot xmlns:xacro="http://www.ros.org/wiki/xacro" name="head_unit">
   <xacro:property name="pi" value="3.14159265359" />
   <link name="head_unit">
@@ -6,8 +6,8 @@
       <origin xyz="0 0 0" rpy="0 0 0" />
       <geometry>
-        <box size="0.0677 0.1120 0.0200" />
+        <box size="0.1268 0.1525 0.0096" />
       </geometry>
       <material name="grey">
-        <color rgba="0.1 0.1 .5 1"/>
+        <color rgba="0.5 0.5 0.5 1"/>
       </material>
     </visual>
@@ -16,21 +16,5 @@
     <parent link="base_link" />
     <child link="head_unit" />
-    <origin xyz="0 0 0.45" rpy="0 0 0" /> <!-- fix height -->
-  </joint>
-  <link name="head_mount">
-    <visual>
-      <origin xyz="0 0 0" rpy="0 0 0" />
-      <geometry>
-        <box size="0.1268 0.1525 0.0096" />
-      </geometry>
-      <material name="silver">
-        <color rgba="129 129 129 1" />
-      </material>
-    </visual>
-  </link>
-  <joint name="head_unit_to_head_mount" type="fixed">
-    <parent link="head_unit" />
-    <child link="head_mount" />
-    <origin xyz="0 0 -0.2159" rpy="0 0 0 " />
+    <origin xyz="0 0 ${platform_h + 0.0096}" rpy="0 0 0" /> <!-- fix height -->
   </joint>
   <link name="t-slot-rod">
@@ -38,7 +22,7 @@
       <origin xyz="0 0 0" rpy="0 0 0" />
       <geometry>
-         <mesh filename="package://head_unit/urdf/meshes/t-slot-rod.stl" scale="1 1 0.2"/>
+         <mesh filename="package://head_unit/urdf/meshes/t-slot-rod.stl" scale="1 1 0.168"/>
       </geometry>
-      <material name="silver" />
+      <material name="grey"/>
     </visual>
   </link>
@@ -46,5 +30,5 @@
     <parent link="head_unit" />
     <child link="t-slot-rod" />
-    <origin xyz="0 0 -0.1065" rpy="0 0 0" />
+    <origin xyz="0 0 ${0.2159/2}" rpy="0 0 0" />
   </joint>
   <xacro:macro name="t-slot-bracket" params="name xyz rpy">
@@ -55,5 +39,5 @@
            <mesh filename="package://head_unit/urdf/meshes/t-slot-bracket.stl" scale="1 1 1"/>
         </geometry>
-        <material name="silver" />
+        <material name="grey" />
       </visual>
     </link>
@@ -64,8 +48,22 @@
     </joint>
   </xacro:macro>
-  <xacro:t-slot-bracket name="bottom-left" xyz="0 0.0191 -0.135" rpy="${pi/2} 0 ${pi/2}" />
-  <xacro:t-slot-bracket name="bottom-right" xyz="0 -0.0191 -0.135" rpy="${pi/2} 0 -${pi/2}" />
-  <xacro:t-slot-bracket name="top-left" xyz="0 0.0191 -0.01" rpy="-${pi/2} 0 ${pi/2}" />
-  <xacro:t-slot-bracket name="top-right" xyz="0 -0.0191 -0.01" rpy="-${pi/2} 0 -${pi/2}" />
+  <xacro:t-slot-bracket name="bottom-left" xyz="0 0.0191 0.004" rpy="${pi/2} 0 ${pi/2}" />
+  <xacro:t-slot-bracket name="bottom-right" xyz="0 -0.0191 0.004" rpy="${pi/2} 0 -${pi/2}" />
+  <xacro:t-slot-bracket name="top-left" xyz="0 0.0191 0.211" rpy="-${pi/2} 0 ${pi/2}" />
+  <xacro:t-slot-bracket name="top-right" xyz="0 -0.0191 0.211" rpy="-${pi/2} 0 -${pi/2}" />
+  <link name="kinect_mount">
+    <visual>
+      <origin xyz="0 0 0" rpy="0 0 0" />
+      <geometry>
+        <box size="0.0677 0.1120 0.0200" />
+      </geometry>
+      <material name="black" />
+    </visual>
+  </link>
+  <joint name="head_unit_to_kinect_mount" type="fixed">
+    <parent link="head_unit" />
+    <child link="kinect_mount" />
+    <origin xyz="-0.013 0 0.2215" rpy="0 0 0 " />
+  </joint>
   <xacro:include filename="../../head_unit/urdf/kinect2.xacro" />
   <xacro:include filename="../../head_unit/urdf/project_tango.xacro" />

File: src/head_unit/urdf/kinect2.xacro (robot description, xacro)
@@ -49,5 +49,5 @@
 -->
   </xacro:macro>
-  <xacro:kinect2_xacro prefix="head_unit" parent="head_unit" rpy="${-pi/2} 0 ${-pi/2}" xyz="0.04 -0.098 0.035" />
+  <xacro:kinect2_xacro prefix="head_unit" parent="head_unit" rpy="${-pi/2} 0 ${-pi/2}" xyz="0.017 -0.098 0.2573" />
  <!--  <xacro:kinect2_xacro prefix="head_unit" parent="head_unit" rpy="0 0 ${pi/2}" xyz="0 0.108 0.07" /> -->
 </robot>

File: src/mobile_base/urdf/mobile_base_mkii.xacro (robot description, xacro)
@@ -9,5 +9,5 @@
       <origin rpy="0 0 ${pi/2}" xyz="0 0 ${platform_h/2}"/>
       <geometry>
-        <mesh filename="package://mobile_base/urdf/meshes/mobile_base_mkii.stl"  scale="1 1 1.18" />
+        <mesh filename="package://mobile_base/urdf/meshes/mobile_base_mkii.stl"  scale="1 1 1" />
       </geometry>
       <material name="black">
@@ -16,19 +16,3 @@
     </visual>
   </link>
-  <link name="base_footprint">
-    <visual>
-      <origin rpy="0 0 0" xyz="0 0 0"/>
-      <geometry>
-        <box size="${platform_l} ${platform_w} 0.001" />
-      </geometry>
-      <material name="black">
-        <color rgb="0 0 0" />
-      </material>
-    </visual>
-  </link>
-  <joint name="base_frame_base_link" type="fixed">
-    <parent link="base_link" />
-    <child link="base_footprint" />
-    <origin xyz="0 0 ${-platform_h/2}" rpy="0 0 0" />
-  </joint>
 </robot>

File: src/navbot/urdf/navbot_mkii.urdf (robot description, URDF)
Before this commit: robot blah, 13 links, 12 joints
Links:
- removed link base_footprint
- removed link head_mount
- added link kinect_mount; visual box size=0.0677 0.1120 0.0200
- link base_link: geometry visual mesh filename=package://mobile_base/urdf/meshes/mobile_base_mkii.stl scale=1 1 1
- link head_unit: geometry visual box size=0.1268 0.1525 0.0096
- link t-slot-rod: geometry visual mesh filename=package://head_unit/urdf/meshes/t-slot-rod.stl scale=1 1 0.168
Joints:
- removed joint base_frame_base_link
- removed joint head_unit_to_head_mount
- added joint head_unit_to_kinect_mount: type fixed, parent head_unit, child kinect_mount, origin xyz=-0.013 0 0.2215 rpy=0 0 0 
- joint base_link_to_head_unit: origin xyz=0 0 0.45 rpy=0 0 0 -> xyz=0 0 0.2509 rpy=0 0 0
- joint head_unit_kinect2_in_joint: origin xyz=0.04 -0.098 0.035 rpy=-1.5707963268 0 -1.5707963268 -> xyz=0.017 -0.098 0.2573 rpy=-1.5707963268 0 -1.5707963268
- joint head_unit_to_t-slot-bracket-bottom-left: origin xyz=0 0.0191 -0.135 rpy=1.5707963268 0 1.5707963268 -> xyz=0 0.0191 0.004 rpy=1.5707963268 0 1.5707963268
- joint head_unit_to_t-slot-bracket-bottom-right: origin xyz=0 -0.0191 -0.135 rpy=1.5707963268 0 -1.5707963268 -> xyz=0 -0.0191 0.004 rpy=1.5707963268 0 -1.5707963268
- joint head_unit_to_t-slot-bracket-top-left: origin xyz=0 0.0191 -0.01 rpy=-1.5707963268 0 1.5707963268 -> xyz=0 0.0191 0.211 rpy=-1.5707963268 0 1.5707963268
- joint head_unit_to_t-slot-bracket-top-right: origin xyz=0 -0.0191 -0.01 rpy=-1.5707963268 0 -1.5707963268 -> xyz=0 -0.0191 0.211 rpy=-1.5707963268 0 -1.5707963268
- joint head_unit_to_t-slot-rod: origin xyz=0 0 -0.1065 rpy=0 0 0 -> xyz=0 0 0.10795 rpy=0 0 0

File: src/navbot/urdf/navbot_mkii.xacro (robot description, xacro)
@@ -1,14 +1,4 @@
 <?xml version="1.0"?>
 <robot xmlns:xacro="http://www.ros.org/wiki/xacro" name="blah">
-<!--  <link name="base_link">
-    <visual>
-      <geometry>
-        <box size="0.001 0.001 0.001"/>
-      </geometry>
-      <material name="black">
-        <color rgba="0 0 0 1" />
-      </material>
-    </visual>
-  </link> -->
   <xacro:include filename="../../mobile_base/urdf/mobile_base_mkii.xacro" />
   <xacro:include filename="../../head_unit/urdf/head_unit_mkii.xacro" />

Commit message: Fixed project tango position in mk ii xacro

File: src/head_unit/urdf/head_unit_mkii.xacro (robot description, xacro)
@@ -6,5 +6,5 @@
       <origin xyz="0 0 0" rpy="0 0 0" />
       <geometry>
-        <box size="0.1268 0.1525 0.0096" />
+        <box size="0.1268 0.1525 0.0095" />
       </geometry>
       <material name="grey">
@@ -16,5 +16,5 @@
     <parent link="base_link" />
     <child link="head_unit" />
-    <origin xyz="0 0 ${platform_h + 0.0096}" rpy="0 0 0" /> <!-- fix height -->
+    <origin xyz="0 0 ${platform_h + 0.014}" rpy="0 0 0" /> <!-- fix height -->
   </joint>
   <link name="t-slot-rod">

File: src/head_unit/urdf/project_tango.xacro (robot description, xacro)
@@ -31,5 +31,5 @@
     <parent link="head_unit" />
     <child link="unity" />
-    <origin xyz="-0.15 0.1 -0.185" rpy="1.22 0 ${-pi/2}" />
+    <origin xyz="0.0875 0.1 0.01" rpy="1.22 0 ${-pi/2}" />
   </joint>
 </robot>

File: src/navbot/urdf/navbot_mkii.urdf (robot description, URDF)
Before this commit: robot blah, 12 links, 11 joints
Links:
- link head_unit: geometry visual box size=0.1268 0.1525 0.0095
Joints:
- joint base_link_to_head_unit: origin xyz=0 0 0.2509 rpy=0 0 0 -> xyz=0 0 0.2553 rpy=0 0 0
- joint head_unit_to_unity: origin xyz=-0.15 0.1 -0.185 rpy=1.22 0 -1.5707963268 -> xyz=0.0875 0.1 0.01 rpy=1.22 0 -1.5707963268
