Commit message: Adding base_footprint to xacro

File: src/mobile_base/urdf/mobile_base_mkii.xacro (robot description, xacro)
@@ -16,3 +16,19 @@
     </visual>
   </link>
+  <link name="base_footprint">
+    <visual>
+      <origin rpy="0 0 0" xyz="0 0 0"/>
+      <geometry>
+        <box size="${platform_l} ${platform_w} 0.001" />
+      </geometry>
+      <material name="black">
+        <color rgb="0 0 0" />
+      </material>
+    </visual>
+  </link>
+  <joint name="base_frame_base_link" type="fixed">
+    <parent link="base_link" />
+    <child link="base_footprint" />
+    <origin xyz="0 0 ${-platform_h/2}" rpy="0 0 0" />
+  </joint>
 </robot>

File: src/navbot/urdf/navbot_mkii.urdf (robot description, URDF)
Before this commit: robot blah, 12 links, 11 joints
Links:
- added link base_footprint; visual box size=0.6096 0.6096 0.001
Joints:
- added joint base_frame_base_link: type fixed, parent base_link, child base_footprint, origin xyz=0 0 -0.12065 rpy=0 0 0

Commit message: Working mobile base mk ii with lidar and odom. Stashing all my tests before serious repo cleanup.

File: src/mobile_base/urdf/mobile_base_mkii.xacro (robot description, xacro)
@@ -16,3 +16,31 @@
     </visual>
   </link>
+  <link name="imu_link">
+    <visual>
+      <origin rpy="0 0 0" xyz="0 0 0"/>
+      <geometry>
+	<box size="0.0305 0.0203 0.0051"/>
+      </geometry>
+    </visual>
+  </link>
+  <joint name="base_link_to_imu_link" type="fixed">
+    <origin rpy="0 0 0" xyz="-0.0238 0 -${platform_h/2 - 0.05}" />
+    <parent link="base_link"/>
+    <child link="imu_link"/>
+  </joint>
+  <link name="neato_laser">
+    <visual>
+      <geometry>
+        <cylinder length="0.018" radius="0.04"/>
+      </geometry>
+      <material name="black">
+        <color rgba="0 0 0 1"/>
+      </material>
+    </visual>
+  </link>
+  <joint name="base_link_to_neato_laser" type="fixed">
+    <origin rpy="0 0 0" xyz="0.102 0  ${platform_h + 0.045}" />
+    <parent link="base_link"/>
+    <child link="neato_laser"/>
+  </joint>
 </robot>

File: src/navbot/urdf/navbot_mkii.urdf (robot description, URDF)
Before this commit: robot blah, 12 links, 11 joints
Links:
- removed link camera_depth_frame
- removed link head_unit
- removed link kinect2_link
- removed link kinect_mount
- removed link phone
- removed link t-slot-bracket-bottom-left
- removed link t-slot-bracket-bottom-right
- removed link t-slot-bracket-top-left
- removed link t-slot-bracket-top-right
- removed link t-slot-rod
- removed link unity
- added link imu_link; visual box size=0.0305 0.0203 0.0051
- added link neato_laser; visual cylinder length=0.018 radius=0.04
Joints:
- removed joint base_link_to_head_unit
- removed joint head_unit_kinect2_in_joint
- removed joint head_unit_to_kinect_mount
- removed joint head_unit_to_t-slot-bracket-bottom-left
- removed joint head_unit_to_t-slot-bracket-bottom-right
- removed joint head_unit_to_t-slot-bracket-top-left
- removed joint head_unit_to_t-slot-bracket-top-right
- removed joint head_unit_to_t-slot-rod
- removed joint head_unit_to_unity
- removed joint kinect2_link_to_camera_depth_frame
- removed joint unity_to_phone
- added joint base_link_to_imu_link: type fixed, parent base_link, child imu_link, origin xyz=-0.0238 0 -0.07065 rpy=0 0 0
- added joint base_link_to_neato_laser: type fixed, parent base_link, child neato_laser, origin xyz=0.102 0  0.2863 rpy=0 0 0

File: src/navbot/urdf/navbot_mkii.xacro (robot description, xacro)
@@ -2,4 +2,5 @@
 <robot xmlns:xacro="http://www.ros.org/wiki/xacro" name="blah">
   <xacro:include filename="../../mobile_base/urdf/mobile_base_mkii.xacro" />
-  <xacro:include filename="../../head_unit/urdf/head_unit_mkii.xacro" />
+<!--  <xacro:include filename="../../head_unit/urdf/head_unit_mkii.xacro" />
+-->
 </robot>
