Commit message: re-adding imu to do localization

File: src/mobile_base/urdf/mobile_base_mkii.urdf (robot description, URDF)
Before this commit: robot mobile_base_mkii, 1 links, 0 joints
Links:
- added link imu_link; visual box size=0.0305 0.0203 0.0051
- added link neato_laser; visual cylinder length=0.018 radius=0.04
- link base_link: geometry visual mesh filename=package://mobile_base/urdf/meshes/mobile_base_mkii.stl scale=1 1 1
Joints:
- added joint base_link_to_imu_link: type fixed, parent base_link, child imu_link, origin xyz=0.0238 0 -0.07065 rpy=0 0 0
- added joint base_link_to_neato_laser: type fixed, parent base_link, child neato_laser, origin xyz=0.102 0  0.2863 rpy=0 0 0

File: src/mobile_base/urdf/mobile_base_mkii.xacro (robot description, xacro)
@@ -25,5 +25,5 @@
   </link>
   <joint name="base_link_to_imu_link" type="fixed">
-    <origin rpy="0 0 0" xyz="-0.0238 0 -${platform_h/2 - 0.05}" />
+    <origin rpy="0 0 0" xyz="0.0238 0 -${platform_h/2 - 0.05}" />
     <parent link="base_link"/>
     <child link="imu_link"/>
